File: hardware/im01.kicad_sch (KiCad schematic)
At the start: 110 parts, among them J1 ПИТАНИЕ 9-30В, J2 COIN, J3 BILL, J4 NANO SIM, J5 U.FL, J6 SWD, Q1 2N7002, Q2 2N7002, SW1 ВЫГРУЗКА, U1 LMR16020, U2 ME6211C33, U3 STM32G030K8T6, U4 FM25L16B, U5 EL817S1(B), U6 EL817S1(B), U7 EG800K-EU, U8 SRV05-4, U9 TXS0102

Commit message: feat(hardware): разводка платы ИМ-01, файлы для JLCPCB, виртуальная модель
Три критичные цепи (антенна, узел SW, путь VBAT) разведены по заданной
геометрии и зафиксированы, остальное — Freerouting; земля досоединяется
по отчёту DRC. Итог: ERC 0 ошибок, DRC 0 нарушений и 0 неподключённых,
сверка платы со схемой — 0 расхождений. fab/: гербер-архив, BOM и CPL
для JLCPCB, PDF схемы и сборочного чертежа, STEP и 3D-вид.
sim/run_final.py — модель всего устройства с окончательными номиналами:
все 5 сценариев проходят (VBAT ≥ 3.53 В, MCU живёт ~50 мс после
пропадания 12 В).

Co-Authored-By: Claude Opus 5 <noreply@anthropic.com>
Parts:
- removed TP7: MODEM_DBG_TX, TestPoint:TestPoint_Pad_D1.0mm, symbol Connector:TestPoint
- removed TP8: MODEM_DBG_RX, TestPoint:TestPoint_Pad_D1.0mm, symbol Connector:TestPoint
Connections:
- net MODEM_DBG_RX: no longer names the net of U7.38 (DBG_RXD)
- net MODEM_DBG_TX: no longer names the net of U7.39 (DBG_TXD)
- no-connect marks 82 -> 84
